File: FlowController/FlowController.sch (EAGLE design)
At the start: 98 parts, among them Q1 G65P06, Q10 G65P06, Q2 G65P06, Q3 G65P06, Q4 G65P06, Q5 G65P06, Q6 G65P06, Q7 G65P06, Q8 G65P06, Q9 G65P06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

Commit message: schematic draft 2
Parts:
- removed C19: 22uF, SparkFun-Capacitors:10UF-1210-50V-20%
- removed C20, C21: 100uF, SparkFun-Capacitors:10UF-1210-50V-20%
- removed C22: 100pF, SparkFun-Capacitors:2.2UF-0805-25V-(+80/-20%)
- removed L1: SRN8040-330M, FlowControllerLib:SRN8040-330M
- removed LED6: (no value), adafruit:LEDCHIPLED_0805
- removed R39: 220k, adafruit:R-US_M0805
- removed R40: 4.7K, adafruit:R-US_M0805
- added C23, C24: 0.1uF, SparkFun-Capacitors:2.2UF-0805-25V-(+80/-20%)
- added D7, D8: BZT52C15-7-F, BZT52C15-7-F:BZT52C15-7-F
- added D9: P6SMB58CA, 1smb59xx_10:1SMB5913BT3G
- added LED7, LED8: (no value), adafruit:LEDCHIPLED_0805
- added Q11, Q12, Q13, Q14: G65P06, FlowControllerLib:G65P06
- added R41, R44: 100k, adafruit:R-US_M0805
- added R42, R43, R45, R46: 4.7k, adafruit:R-US_M0805
- added R47: 100, SparkFun-Resistors:0.05OHM-2512-3W-1%
- added R48, R49: 4.7K, adafruit:R-US_M0805
- added U8, U9: TCMT1100SOP-4L_TC-M, FlowControllerLib:TCMT1100SOP-4L_TC-M
- U7: value LTC3630EMSETRPBF -> ACZRC5370B-G; device FlowControllerLib:LTC3630EMSETRPBF -> FlowControllerLib:ACZRC5370B-G
Connections:
- removed net D8: J1.5
- removed net D9: J1.4
- removed net N$21: R5.1, U2.C
- removed net N$39: C22.1, R39.2, U7.ISET
- removed net N$76: LED6.C, R40.2
- removed net POWER_DIODE_OUT+: C19.1, I2.IP+, U7.VIN
- removed net SW: L1.2, U7.SW
- new net BATTERY_OUT+: I2.IP-, R28.2
- new net BATTERY_OUT_I_SENSE+: I2.IP+, Q11.D, Q13.D
- new net EXT_BUS_FUSED+: I1.IP+
- new net G_PRECHARGE_4: R45.1, R49.1, U9.C
- new net G_SWITCH_3: R12.1, R5.1, U2.C
- new net G_SWITCH_4: R42.1, R48.1, U8.C
- new net N$10: C24.1, D8.A, Q13.G, Q14.G, R44.1, R45.2
- new net N$12: R46.1, U9.A
- new net N$13: Q14.D, R47.1
- new net N$15: LED7.C, R48.2
- new net N$17: LED8.C, R49.2
- new net N$7: C23.1, D7.A, Q11.G, Q12.G, R41.1, R42.2
- new net N$9: R43.1, U8.A
- new net PRECHARGE_4: J1.6, R46.2
- new net SWITCH_4: J1.5, R43.2
- new net S_PRECHARGE_4: C24.2, D8.C, LED8.A, Q13.S, Q14.S, R44.2
- new net S_SWITCH_3: C2.2, D2.C, LED3.A, Q2.S, Q5.S, R8.2
- net +5V: no longer C20.1, C21.1, L1.1, LED6.A, U7.VFB
- net CURRENT_LIMIT_ENABLE: now also J1.4; no longer J1.6
- net EXT_BUS+: no longer I1.IP+
- net FLOW_BUS+: now also Q12.D, R47.2; no longer I2.IP-, R20.2, R28.2
- net GND: now also D9.A, U7.2, U8.C_2, U8.E, U9.C_2, U9.E; no longer C19.2, C20.2, C21.2, C22.2, R39.1, R40.1, U7.GND, U7.GND_2, U7.GND_3, U7.GND_4, U7.VPRG2
- net G_SWITCH_2: no longer R12.1
- net SS: no longer U7.SS, U7.VPRG1
- net S_SWITCH_2: no longer LED3.A
- net S_SWITCH_4: now also C23.2, D7.C, LED7.A, Q11.S, Q12.S, R41.2; no longer C2.2, D2.C, Q2.S, Q5.S, R8.2
- net WORM_BUS+: now also D9.C, R20.2, U7.1
Other:
- note added: "BF1 58V FUSE"
- note removed: "5V POWER"
- moved on the sheet: C10, C11, C12, C13, C14, C15, C16, C17, C18, C6, C7, C8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
