File: FlowController/FlowControllerFinal.brd (EAGLE design)
At the start: 188 x 65 mm, 97 parts, among them IC1 LM358_DIP, IC2 LM358_DIP, U18 FAN7081M-GF085, U19 STH140N8F7-2, U2 FAN7081M-GF085, U20 STH140N8F7-2, U21 CDBM1100-G, U22 CDBM1100-G, U23 FAN7081M-GF085, U24 STH140N8F7-2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

Commit message: Finalized board and CAM files
Parts:
- removed IC1, IC2: LM358_DIP, IC_Linear:DIP826W53P254L959H508Q8B
- added U4, U5: LM358PSR, FlowControllerLib:PS8
- C16: value 22uF -> 10uF
- C17: value 2.2uF -> 10uF
- R16, R2, R5, R8: value 10k -> 10K
- R38: device adafruit:M0805 -> SparkFun-Resistors:2512
- moved R38 136.6 mm to (67.6, 47.4)
- moved C10 134.0 mm to (24.5, 38.9)
- moved C11 134.0 mm to (27.6, 38.9)
- moved C12 134.0 mm to (50.9, 44.2)
- moved C13 134.0 mm to (55.4, 42.1)
- moved C14 134.0 mm to (64.2, 47.9)
- moved C15 134.0 mm to (62.8, 50.9)
- moved C16 134.0 mm to (72.9, 50.8)
- moved C18 134.0 mm to (47.1, 51.7)
- moved C2 134.0 mm to (126.1, 62.1)
- moved C22 134.0 mm to (62.1, 31.0)
- moved C23 134.0 mm to (153.1, 15.8)
- moved C24 134.0 mm to (53.4, 24.1)
- moved C25 134.0 mm to (143.1, 15.4)
- moved C26 134.0 mm to (67.1, 13.3)
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Connections:
- net +5V: now also U4.8, U5.8; no longer IC1.8, IC2.8
- net CHARGER+: now also R38.P$2; no longer R38.2
- net GND: now also U4.4, U5.4; no longer IC1.4, IC2.4
- net SENSE: now also R38.P$1; no longer R38.1
- net V_SENSE_1: now also U5.1, U5.2; no longer IC1.1, IC1.3
- net V_SENSE_1_PRE: now also U5.3; no longer IC1.2
- net V_SENSE_2: now also U5.6, U5.7; no longer IC1.6, IC1.7
- net V_SENSE_2_PRE: now also U5.5; no longer IC1.5
- net V_SENSE_3: now also U4.5; no longer IC2.6, IC2.7
- net V_SENSE_3_PRE: now also U4.6, U4.7; no longer IC2.5
Routing:
- net +5V: track 181.8 -> 163.9 mm
- net V_SENSE_1: track 32.9 -> 26.1 mm, vias 1 -> 2
- net V_SENSE_3_PRE: track 115.8 -> 121.7 mm, vias 1 -> 2
- net GND: track 118.3 -> 113.2 mm, vias 130 -> 132
- net V_SENSE_3: track 20.4 -> 17.0 mm
- net SENSE: track 6.33 -> 8.88 mm
- net CURRENT_LIMIT_ENABLE: track 39.6 -> 41.2 mm
- net V_SENSE_1_PRE: track 98.3 -> 97.3 mm, vias 1 -> 2
- net CHARGER+: track 16.1 -> 15.8 mm, vias 44 -> 43
- net V_SENSE_2_PRE: track 116.7 -> 116.9 mm, vias 3 -> 4
Other:
- board size 188 x 65 mm -> 188 x 73 mm
