File: FlowController/FlowControllerFinal.sch (EAGLE design)
At the start: 97 parts, among them IC1 LM358_DIP, IC2 LM358_DIP, U18 FAN7081M-GF085, U19 STH140N8F7-2, U2 FAN7081M-GF085, U20 STH140N8F7-2, U21 CDBM1100-G, U22 CDBM1100-G, U23 FAN7081M-GF085, U24 STH140N8F7-2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

Commit message: Finalized board and CAM files
Parts:
- removed IC1, IC2: LM358_DIP, IC_Linear:LM358_DIP
- added U4, U5: LM358PSR, FlowControllerLib:LM358PSR
- C16: value 22uF -> 10uF
- C17: value 2.2uF -> 10uF
- R16, R2, R5, R8: value 10k -> 10K
- R38: device adafruit:R-US_M0805 -> SparkFun-Resistors:0.05OHM-2512-3W-1%
Connections:
- net +5V: now also U4.VCC, U5.VCC; no longer IC1.V+, IC2.V+
- net GND: now also U4.GND, U5.GND; no longer IC1.V-, IC2.V-
- net V_SENSE_1: now also U5.1IN-, U5.1OUT; no longer IC1.+IN1, IC1.OUT1
- net V_SENSE_1_PRE: now also U5.1IN+; no longer IC1.-IN1
- net V_SENSE_2: now also U5.2IN-, U5.2OUT; no longer IC1.-IN2, IC1.OUT2
- net V_SENSE_2_PRE: now also U5.2IN+; no longer IC1.+IN2
- net V_SENSE_3: now also U4.2IN+; no longer IC2.-IN2, IC2.OUT2
- net V_SENSE_3_PRE: now also U4.2IN-, U4.2OUT; no longer IC2.+IN2
Other:
- moved on the sheet: C17, C18
